Commit message: Removed all links except for the body. Got it to load in Gazebo.

File: Prius_urdf/prius.urdf (robot description, URDF)
Before this commit: robot car, 17 links, 16 joints
Links:
- removed link chassis_floor
- removed link front_axle
- removed link front_left_wheel_center
- removed link front_right_wheel_center
- removed link left_hub
- removed link left_tie_rod_arm
- removed link left_wheel
- removed link left_wheel_rear
- removed link rear_axle
- removed link rear_left_wheel_center
- removed link rear_right_wheel_center
- removed link right_hub
- removed link right_tie_rod_arm
- removed link right_wheel
- removed link right_wheel_rear
- removed link tie_rod
- link body: geometry collision mesh filename=prius.dae scale=1 1 1; visual mesh filename=prius.dae scale=1 1 1
Joints:
- removed joint body
- removed joint chassis_floor_axle
- removed joint chassis_rear_axle
- removed joint front_left_suspension
- removed joint front_right_suspension
- removed joint left_hub
- removed joint left_pin
- removed joint left_wheel_joint
- removed joint rear_left_suspension
- removed joint rear_left_wheel_joint
- removed joint rear_right_suspension
- removed joint rear_right_wheel_joint
- removed joint right_hub
- removed joint right_pin
- removed joint right_wheel_joint
- removed joint steering

Commit message: Got left_tie_rod_arm to work.

File: Prius_urdf/prius.urdf (robot description, URDF)
Before this commit: robot car, 1 links, 0 joints
Links:
- added link front_axle, mass 5.42793634; collision box size=0.061842105 1.051315789 0.030921; visual box size=0.061842105 1.051315789 0.030921
- added link left_tie_rod_arm, mass 1.58382895; visual box size=0.061842105 0.140955396 0.030921; visual box size=0.204636598 0.061842105 0.030921
Joints:
- added joint body: type fixed, parent front_axle, child body, origin xyz=0 0 0, axis 0 0 1
- added joint steering: type revolute, parent front_axle, child left_tie_rod_arm, origin xyz=0 0.494736842 0, axis 0 0 1, limit lower=-0.401425728 upper=0.5 effort=100 velocity=1

Commit message: Added left_pin joint and tie rod.

File: Prius_urdf/prius.urdf (robot description, URDF)
Before this commit: robot car, 3 links, 2 joints
Links:
- added link tie_rod, mass 4.53748175; visual box size=0.061842105 0.878847118 0.030921
- link front_axle: mass 5.42793634 -> None; geometry visual box size=0.061842105 1.051315789 0.030921
Joints:
- added joint left_pin: type continuous, parent left_tie_rod_arm, child tie_rod, origin xyz=-0.172468672 -0.086234287 0, axis 0 0 1, limit lower=-3.1416 upper=3.1416 effort=100 velocity=1

Commit message: Added right_tie_rod_arm link and right_pin joint.

File: Prius_urdf/prius.urdf (robot description, URDF)
Before this commit: robot car, 4 links, 3 joints
Links:
- added link right_tie_rod_arm, mass 1.58382895; visual box size=0.061842105 0.140955396 0.030921; visual box size=0.204636598 0.061842105 0.030921
Joints:
- added joint right_pin: type continuous, parent tie_rod, child right_tie_rod_arm, origin xyz=0 -0.817005012 0, axis 0 0 1, limit lower=-3.1416 upper=3.1416 effort=100 velocity=100
- joint left_pin: limit lower=-3.1416 upper=3.1416 effort=100 velocity=1 -> lower=-3.1416 upper=3.1416 effort=100 velocity=100
- joint steering: limit lower=-0.401425728 upper=0.5 effort=100 velocity=1 -> lower=-0.401425728 upper=0.5 effort=100 velocity=100
